File: usbcan_20190426.brd (EAGLE design)
At the start: 40 x 50 mm, 45 parts, among them J1 8P8C-LED, J2 MICRO-USB-RECEPTACLE47589-0001, J3 MA04-1, J4 MA02-2, U1 STM32F302C, U2 NCV7351D1E, U3 SI8621AB-B-IS, U4 AP2127N-3.3TRG1, U5 78L05F, X1 CSTCE8M00G55

Commit message: value update
Parts:
- C3, C4: value (none) -> 100n
- D1: value (none) -> GREEN
- D2: value (none) -> YELLOW
- D3: value (none) -> RED
- R1: value (none) -> 1k
- R2: value (none) -> 470
Changed lines of the file:
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@@
 <?xml version="1.0" encoding="utf-8"?>
 <!DOCTYPE eagle SYSTEM "eagle.dtd">
-<eagle version="9.3.0">
+<eagle version="9.6.2">
 <drawing>
 <settings>
@@
 </autorouter>
 <elements>
-<element name="C3" library="rcl" library_urn="urn:adsk.eagle:library:334" package="C0603" package3d_urn="urn:adsk.eagle:package:23616/2" value="" x="1.75" y="35.5" smashed="yes" rot="MR270">
+<element name="C3" library="rcl" library_urn="urn:adsk.eagle:library:334" package="C0603" package3d_urn="urn:adsk.eagle:package:23616/2" value="100n" x="1.75" y="35.5" smashed="yes" rot="MR270">
 <attribute name="NAME" x="0.635" y="37.365" size="1.016" layer="26" font="vector" rot="MR90"/>
 <attribute name="SPICEPREFIX" value="C" x="43.66" y="-1.33" size="1.778" layer="28" rot="MR270" display="off"/>
 <attribute name="VALUE" x="3.655" y="36.135" size="1.27" layer="28" rot="MR270"/>
 </element>
-<element name="R1" library="rcl" library_urn="urn:adsk.eagle:library:334" package="R0603" package3d_urn="urn:adsk.eagle:package:23555/3" value="" x="8.75" y="35.25" smashed="yes" rot="R270">
+<element name="R1" library="rcl" library_urn="urn:adsk.eagle:library:334" package="R0603" package3d_urn="urn:adsk.eagle:package:23555/3" value="1k" x="8.75" y="35.25" smashed="yes" rot="R270">
 <attribute name="NAME" x="10.365" y="36.865" size="1.016" layer="25" font="vector" rot="R90"/>
 <attribute name="SPICEPREFIX" value="R" x="-33.16" y="-5.39" size="1.778" layer="27" rot="R270" display="off"/>
 <attribute name="VALUE" x="6.845" y="35.885" size="1.27" layer="27" rot="R270"/>
 </element>
-<element name="R2" library="rcl" library_urn="urn:adsk.eagle:library:334" package="R0603" package3d_urn="urn:adsk.eagle:package:23555/3" value="" x="20.25" y="30.5" smashed="yes" rot="MR180">
+<element name="R2" library="rcl" library_urn="urn:adsk.eagle:library:334" package="R0603" package3d_urn="urn:adsk.eagle:package:23555/3" value="470" x="20.25" y="30.5" smashed="yes" rot="MR180">
 <attribute name="NAME" x="18.615" y="29.365" size="1.016" layer="26" font="vector" rot="MR180"/>
 <attribute name="SPICEPREFIX" value="R" x="64.7" y="72.41" size="1.778" layer="28" rot="MR180" display="off"/>
@@
 <attribute name="SPICEPREFIX" value="C" x="34" y="36.25" size="1.778" layer="27" rot="R180" display="off"/>
 </element>
-<element name="C4" library="rcl" library_urn="urn:adsk.eagle:library:334" package="C0603" package3d_urn="urn:adsk.eagle:package:23616/2" value="" x="10.5" y="32.25" smashed="yes" rot="MR180">
+<element name="C4" library="rcl" library_urn="urn:adsk.eagle:library:334" package="C0603" package3d_urn="urn:adsk.eagle:package:23616/2" value="100n" x="10.5" y="32.25" smashed="yes" rot="MR180">
 <attribute name="NAME" x="11.385" y="33.385" size="1.016" layer="26" font="vector" rot="MR0"/>
 <attribute name="SPICEPREFIX" value="C" x="10.5" y="32.25" size="1.778" layer="28" rot="MR180" display="off"/>
@@
 <attribute name="NAME" x="8.865" y="23.635" size="1.016" layer="25" font="vector"/>
 </element>
-<element name="D1" library="led" library_urn="urn:adsk.eagle:library:259" package="CHIPLED_0805" package3d_urn="urn:adsk.eagle:package:15821/2" value="" x="2.75" y="26" smashed="yes" rot="R90">
+<element name="D1" library="led" library_urn="urn:adsk.eagle:library:259" package="CHIPLED_0805" package3d_urn="urn:adsk.eagle:package:15821/2" value="GREEN" x="2.75" y="26" smashed="yes" rot="R90">
 <attribute name="NAME" x="3.52" y="19.98" size="1.016" layer="25" font="vector" rot="R180"/>
 <attribute name="VALUE" x="4.02" y="28.54" size="1.27" layer="27" rot="R180"/>
 </element>
-<element name="D2" library="led" library_urn="urn:adsk.eagle:library:259" package="CHIPLED_0805" package3d_urn="urn:adsk.eagle:package:15821/2" value="" x="2.75" y="23.5" smashed="yes" rot="R90">
+<element name="D2" library="led" library_urn="urn:adsk.eagle:library:259" package="CHIPLED_0805" package3d_urn="urn:adsk.eagle:package:15821/2" value="YELLOW" x="2.75" y="23.5" smashed="yes" rot="R90">
 <attribute name="NAME" x="3.52" y="18.48" size="1.016" layer="25" font="vector" rot="R180"/>
 <attribute name="VALUE" x="4.02" y="26.04" size="1.27" layer="27" rot="R180"/>
 </element>
-<element name="D3" library="led" library_urn="urn:adsk.eagle:library:259" package="CHIPLED_0805" package3d_urn="urn:adsk.eagle:package:15821/2" value="" x="2.75" y="21" smashed="yes" rot="R90">
+<element name="D3" library="led" library_urn="urn:adsk.eagle:library:259" package="CHIPLED_0805" package3d_urn="urn:adsk.eagle:package:15821/2" value="RED" x="2.75" y="21" smashed="yes" rot="R90">
 <attribute name="NAME" x="3.52" y="16.98" size="1.016" layer="25" font="vector" rot="R180"/>
 <attribute name="VALUE" x="4.02" y="23.54" size="1.27" layer="27" rot="R180"/>
